Commit message: Update 4leggedRobot.urdf

File: src/4leggedRobot.urdf (robot description, URDF)
Before this commit: robot materials, 17 links, 16 joints
Links:
- link base_link: mass 1.843 -> 1.248; geometry collision mesh filename=package://STL_simulation/base_link.stl; visual mesh filename=package://STL_simulation/base_link.stl
- link coxa_BL: mass 0.178 -> 0.09; geometry visual mesh filename=package://STL_simulation/coxa_bl.stl
- link coxa_BR: mass 0.178 -> 0.09; geometry visual mesh filename=package://STL_simulation/coxa_br.stl
- link coxa_FL: mass 0.0827 -> 0.075; geometry visual mesh filename=package://STL_simulation/coxa_fl.stl
- link coxa_FR: mass 0.0827 -> 0.075; geometry visual mesh filename=package://STL_simulation/coxa_fr.stl
- link femur_BL: mass 0.1784 -> 0.085; geometry visual mesh filename=package://STL_simulation/femur_bl.stl
- link femur_BR: mass 0.1784 -> 0.085; geometry visual mesh filename=package://STL_simulation/femur_br.stl
- link femur_FL: mass 0.1784 -> 0.084; geometry visual mesh filename=package://STL_simulation/femur_fl.stl
- link femur_FR: mass 0.1784 -> 0.084; geometry visual mesh filename=package://STL_simulation/femur_fr.stl
- link foot_FL: mass 0.00044 -> 0.0044
- link tibia_BL: mass 0.039 -> 0.034; geometry visual mesh filename=package://STL_simulation/tibia_bl.stl
- link tibia_BR: mass 0.039 -> 0.034; geometry visual mesh filename=package://STL_simulation/tibia_br.stl
- link tibia_FL: mass 0.0377 -> 0.034; geometry visual mesh filename=package://STL_simulation/tibia_fl.stl
- link tibia_FR: mass 0.0377 -> 0.034; geometry visual mesh filename=package://STL_simulation/tibia_fr.stl
Joints:
- joint coxaF_BL: origin xyz=-0.095 0.04 0 -> xyz=0 0.04 0
- joint coxaF_BR: origin xyz=-0.095 -0.04 0 -> xyz=0 -0.04 0
- joint coxaF_FL: origin xyz=0.095 0.04 0 -> xyz=0 0.04 0
- joint coxaF_FR: origin xyz=0.095 -0.04 0 -> xyz=0 -0.04 0
- joint femurF_BL: origin xyz=0 0.04 0 -> xyz=-0.095 0 0
- joint femurF_BR: origin xyz=0 -0.04 0 -> xyz=-0.095 0 0
- joint femurF_FL: origin xyz=0 0.04 0 -> xyz=0.095 0 0
- joint femurF_FR: origin xyz=0 -0.04 0 -> xyz=0.095 0 0
- joint footF_BL: origin xyz=0 0 -0.1 -> xyz=0 0.04 -0.1
- joint footF_BR: origin xyz=0 0 -0.1 -> xyz=0 -0.04 -0.1
- joint footF_FL: origin xyz=0 0 -0.10 -> xyz=0 0.04 -0.1
- joint footF_FR: origin xyz=0 0 -0.10 -> xyz=0 -0.04 -0.1
- joint tibiaF_FL: origin xyz=0 0 -0.10 -> xyz=0 0 -0.1
- joint tibiaF_FR: origin xyz=0 0 -0.10 -> xyz=0 0 -0.1
